File: JTAG-adapter.kicad_pcb (KiCad board)
At the start: 2 copper layers, 50 x 35 mm, 16 parts, among them J1 20-pin JTAG 0.1", J2 10-pin ST-Link 0.1", J3 20-pin JTAG 0.1", J4 10-pin JTAG 0.05", J5 10-pin ST-Link 0.1", J6 6-pin Tag-Connect, U1 MIC5504-3.3YM5

Commit message: WIP commit
Parts:
- removed J2: 10-pin ST-Link 0.1", Connector_IDC:IDC-Header_2x05_P2.54mm_Vertical
- removed JP7: ~, Connector_PinHeader_2.54mm:PinHeader_1x02_P2.54mm_Vertical
- added G***: LOGO, project_footprints:Logo_Endian_Symbol_8x9mm, F.Cu at (21.8, 29.0)
- JP1, JP2, JP4, JP6: footprint Connector_PinHeader_2.54mm:PinHeader_1x02_P2.54mm_Vertical -> Jumper:SolderJumper-2_P1.3mm_Bridged_RoundedPad1.0x1.5mm; moved to B.Cu
- JP3: footprint Connector_PinHeader_2.54mm:PinHeader_1x02_P2.54mm_Vertical -> Jumper:SolderJumper-2_P1.3mm_Open_RoundedPad1.0x1.5mm; moved to B.Cu
- moved JP2 136.3 mm to (4.00, 3.00), turned to 0 degrees
- moved JP1 120.8 mm to (13.0, 3.00), turned to 180 degrees
- moved J4 107.7 mm to (21.0, 16.0), turned to 0 degrees
- moved JP6 105.8 mm to (27.3, 12.3), turned to 270 degrees
- moved J5 104.4 mm to (30.0, 22.6)
- moved C2 103.7 mm to (31.8, 27.0), turned to 0 degrees
- moved J6 99.3 mm to (28.0, 4.00), turned to 270 degrees
- moved JP4 97.7 mm to (14.0, 33.0), turned to 0 degrees
- moved JP3 96.9 mm to (33.0, 26.0), turned to 180 degrees
- moved JP5 96.3 mm to (28.2, 28.8), turned to 0 degrees
- moved U1 95.5 mm to (31.8, 30.0)
- moved J1 93.9 mm to (11.0, 6.07)
- moved J3 93.6 mm to (5.00, 6.07)
- moved C1 90.7 mm to (31.8, 33.0), turned to 180 degrees
Connections:
- J3 pad 1: Net-(J3-Pad1) -> /VCC
- J3 pad 10: /SWDCLK -> GND
- J3 pad 11: GND -> /RTCK
- J3 pad 12: /RTCK -> GND
- J3 pad 13: GND -> /SWIM
- J3 pad 14: /SWIM -> GND
- J3 pad 15: GND -> /nRESET
- J3 pad 16: /nRESET -> GND
- J3 pad 17: GND -> /DBGRQ
- J3 pad 18: /DBGRQ -> GND
- J3 pad 19: GND -> /DBACK
- J3 pad 2: /VCC -> Net-(J3-Pad2)
- J3 pad 20: /DBACK -> GND
- J3 pad 3: GND -> /TRST
- J3 pad 4: /TRST -> GND
- J3 pad 5: GND -> /TDI
- J3 pad 6: /TDI -> GND
- J3 pad 7: GND -> /SWDIO
- J3 pad 8: /SWDIO -> GND
- J3 pad 9: GND -> /SWDCLK
- J5 pad 1: /SWDCLK -> /nRESET
- J5 pad 2: /nRESET -> /SWDCLK
- J5 pad 3: /SWDIO -> /SWIM
- J5 pad 4: /SWIM -> /SWDIO
- JP2 pad 1: Net-(J3-Pad1) -> Net-(J3-Pad2)
- JP3 pad 1: +5V -> /ST-Link_3V3
- JP3 pad 2: /VCC -> +3V3
Routing:
- net /VCC: track 0.00 -> 83.6 mm, vias 0 -> 1
- net /SWIM: track 0.00 -> 51.0 mm, vias 0 -> 3
- net /nRESET: track 0.00 -> 49.2 mm, vias 0 -> 1
- net /SWDCLK: track 0.00 -> 46.9 mm, vias 0 -> 3
- net /SWDIO: track 0.00 -> 44.4 mm, vias 0 -> 2
- net +5V: track 0.00 -> 41.5 mm, vias 0 -> 2
- net /TDI: track 0.00 -> 30.0 mm
- net /ST-Link_3V3: track 0.00 -> 15.2 mm
- net /DBACK: track 0.00 -> 11.0 mm
- net +3V3: track 0.00 -> 6.72 mm, vias 0 -> 1
- net /TRST: track 0.00 -> 6.00 mm
- net /RTCK: track 0.00 -> 6.00 mm
- net /DBGRQ: track 0.00 -> 6.00 mm
- net /ST-Link_5V: track 0.00 -> 5.56 mm
- net Net-(J3-Pad2): track 0.00 -> 3.44 mm
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- added copper zone on B.Cu, net GND
- added copper zone on F.Cu, net GND
Other:
- board size 50 x 35 mm -> 35 x 35 mm
- net class Default: via_dia 0.8 -> 0.6; via_drill 0.4 -> 0.3
- board text added: "Debugger adapter V1.0"
- board text added: "EN VCC"
